File: pcb/charliewatch.brd (EAGLE design)
At the start: 33 x 33 mm, 85 parts, among them U2 CC430F5137IRGZR, X1 CRYSTALS-NOGND-IQXC-25, X2 FA-128

Commit message: as orderd v0.1
Parts:
- moved JP1 0.77 mm to (18.0, 27.0), flipped to the bottom
Other:
- board text added: "10"
- board text added: "11"
- board text added: "v0.1"
- board text removed: "00"
- board text removed: "0A"
- board text removed: "0B"
Changed lines of the file:
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@@
 <plain>
 <circle x="25.4" y="25.4" radius="16.51" width="0.4064" layer="20"/>
-<text x="39.37" y="19.05" size="0.8128" layer="26" font="vector" rot="MR330">https://trmm.net/Charliewatch</text>
-<text x="26.035" y="37.1475" size="1.016" layer="25" font="vector">00</text>
-<text x="29.21" y="36.195" size="1.016" layer="25" font="vector">01</text>
-<text x="34.29" y="32.0675" size="1.016" layer="25" font="vector">02</text>
-<text x="36.5125" y="26.035" size="1.016" layer="25" font="vector">03</text>
-<text x="35.56" y="20.32" size="1.016" layer="25" font="vector">04</text>
-<text x="31.75" y="15.875" size="1.016" layer="25" font="vector">05</text>
-<text x="23.1775" y="13.0175" size="1.016" layer="25" font="vector">06</text>
-<text x="17.4625" y="15.5575" size="1.016" layer="25" font="vector">07</text>
-<text x="13.97" y="20.32" size="1.016" layer="25" font="vector">08</text>
-<text x="12.7" y="26.035" size="1.016" layer="25" font="vector">09</text>
-<text x="14.9225" y="32.0675" size="1.016" layer="25" font="vector">0A</text>
-<text x="20.32" y="36.195" size="1.016" layer="25" font="vector">0B</text>
-<text x="19.685" y="18.7325" size="0.6096" layer="25" font="vector" rot="R180">GND</text>
-<text x="20.955" y="21.9075" size="0.6096" layer="25" font="vector" rot="R90">TEST</text>
-<text x="20.955" y="24.4475" size="0.6096" layer="25" font="vector" rot="R90">VCC</text>
-<text x="20.955" y="27.305" size="0.6096" layer="25" font="vector" rot="R90">RX</text>
-<text x="20.955" y="29.845" size="0.6096" layer="25" font="vector" rot="R90">TX</text>
-<text x="20.955" y="32.0675" size="0.6096" layer="25" font="vector" rot="R90">RST</text>
-<text x="33.02" y="24.13" size="0.4064" layer="25" font="vector">RF+</text>
-<text x="33.3375" y="24.765" size="0.4064" layer="25" font="vector">RF-</text>
+<text x="38.6715" y="19.939" size="0.8128" layer="26" font="vector" rot="MR330">https://trmm.net/Charliewatch</text>
+<text x="28.1305" y="35.8775" size="1.778" layer="25" font="vector">01</text>
+<text x="32.8295" y="32.1945" size="1.778" layer="25" font="vector">02</text>
+<text x="35.6235" y="26.0985" size="1.778" layer="25" font="vector">03</text>
+<text x="35.052" y="20.447" size="1.778" layer="25" font="vector">04</text>
+<text x="31.623" y="15.6845" size="1.778" layer="25" font="vector">05</text>
+<text x="26.2255" y="12.954" size="1.778" layer="25" font="vector">06</text>
+<text x="20.2565" y="13.843" size="1.778" layer="25" font="vector">07</text>
+<text x="15.113" y="17.272" size="1.778" layer="25" font="vector">08</text>
+<text x="12.7635" y="22.86" size="1.778" layer="25" font="vector">09</text>
+<text x="13.462" y="28.5115" size="1.778" layer="25" font="vector">10</text>
+<text x="20.066" y="35.4965" size="1.778" layer="25" font="vector">11</text>
+<text x="19.431" y="21.463" size="0.6096" layer="25" font="vector" rot="R270">GND</text>
+<text x="20.1295" y="22.225" size="0.6096" layer="25" font="vector" rot="R90">TEST</text>
+<text x="20.066" y="24.892" size="0.6096" layer="25" font="vector" rot="R90">VCC</text>
+<text x="20.1295" y="27.686" size="0.6096" layer="25" font="vector" rot="R90">RX</text>
+<text x="20.066" y="30.353" size="0.6096" layer="25" font="vector" rot="R90">TX</text>
+<text x="20.066" y="32.385" size="0.6096" layer="25" font="vector" rot="R90">RST</text>
+<text x="32.766" y="23.622" size="0.6096" layer="25" font="vector">RF+</text>
+<text x="33.02" y="24.511" size="0.6096" layer="25" font="vector">RF-</text>
 <rectangle x1="23.65501875" y1="14.76375" x2="23.71598125" y2="14.82725" layer="25"/>
 <rectangle x1="26.95701875" y1="14.76375" x2="27.08148125" y2="14.82725" layer="25"/>
@@
 <rectangle x1="24.98851875" y1="19.52625" x2="25.75051875" y2="19.58975" layer="25"/>
 <rectangle x1="24.98851875" y1="19.58975" x2="25.75051875" y2="19.65325" layer="25"/>
+<text x="23.749" y="33.655" size="1.27" layer="25" font="vector">v0.1</text>
 </plain>
 <attributes>
@@
 </element>
 <element name="R1" library="rcl" package="R0603" value="75k" x="27.94" y="31.115" smashed="yes" rot="R180">
-<attribute name="NAME" x="30.48" y="32.0675" size="0.6096" layer="25" rot="R180"/>
+<attribute name="NAME" x="30.48" y="32.0675" size="0.4064" layer="25" rot="R180"/>
 <attribute name="VALUE" x="28.575" y="33.02" size="0.6096" layer="27" rot="R180"/>
 </element>
 <element name="L1" library="rcl" package="R0603" value="" x="31.75" y="29.845" smashed="yes">
-<attribute name="NAME" x="33.3375" y="29.845" size="0.6096" layer="25"/>
+<attribute name="NAME" x="33.3375" y="29.845" size="0.4064" layer="25"/>
 <attribute name="VALUE" x="31.115" y="27.94" size="1.27" layer="27"/>
 </element>
 <element name="R2" library="rcl" package="R0603" value="56k" x="31.75" y="27.94" smashed="yes" rot="R180">
-<attribute name="NAME" x="34.29" y="28.575" size="0.6096" layer="25" rot="R180"/>
+<attribute name="NAME" x="33.9725" y="28.2575" size="0.4064" layer="25" rot="R180"/>
 <attribute name="VALUE" x="32.385" y="29.845" size="0.6096" layer="27" rot="R180"/>
 </element>
 <element name="C1" library="resistor" package="C0603" value="" x="32.0675" y="22.86" smashed="yes">
-<attribute name="NAME" x="33.655" y="22.86" size="0.6096" layer="25"/>
+<attribute name="NAME" x="33.655" y="22.6695" size="0.4064" layer="25"/>
 <attribute name="VALUE" x="31.4325" y="20.955" size="1.27" layer="27"/>
 </element>
 <element name="C2" library="resistor" package="C0603" value="" x="31.75" y="26.035" smashed="yes">
-<attribute name="NAME" x="33.3375" y="26.035" size="0.6096" layer="25"/>
+<attribute name="NAME" x="33.274" y="25.8445" size="0.4064" layer="25"/>
 <attribute name="VALUE" x="31.115" y="24.13" size="1.27" layer="27"/>
 </element>
 <element name="C3" library="resistor" package="C0603" value="" x="20.955" y="19.3675" smashed="yes" rot="R270">
-<attribute name="NAME" x="21.9075" y="17.78" size="0.6096" layer="25"/>
+<attribute name="NAME" x="20.701" y="20.955" size="0.4064" layer="25"/>
 <attribute name="VALUE" x="19.05" y="20.0025" size="1.27" layer="27" rot="R270"/>
 </element>
@@
 </element>
 <element name="C4" library="resistor" package="C0603" value="19pf" x="28.8925" y="20.32" smashed="yes" rot="R180">
-<attribute name="NAME" x="27.305" y="20.6375" size="0.6096" layer="25" rot="R180"/>
+<attribute name="NAME" x="27.305" y="20.6375" size="0.4064" layer="25" rot="R180"/>
 <attribute name="VALUE" x="29.5275" y="22.225" size="1.27" layer="27" rot="R180"/>
 </element>
 <element name="C5" library="resistor" package="C0603" value="19pf" x="32.0675" y="20.955" smashed="yes">
-<attribute name="NAME" x="33.655" y="21.2725" size="0.6096" layer="25"/>
+<attribute name="NAME" x="33.655" y="20.8915" size="0.4064" layer="25"/>
 <attribute name="VALUE" x="31.4325" y="19.05" size="1.27" layer="27"/>
 </element>
@@
 <attribute name="VALUE" x="35.3145" y="16.863584375" size="1.6764" layer="28" font="vector" rot="MR330"/>
 </element>
-<element name="JP1" library="adafruit" package="1X06-BIGLOCK" value="" x="18.7325" y="26.67" smashed="yes" rot="R90">
-<attribute name="VALUE" x="21.9075" y="19.05" size="1.27" layer="27" rot="R90"/>
+<element name="JP1" library="adafruit" package="1X06-BIGLOCK" value="" x="18.034" y="26.9875" smashed="yes" rot="MR90">
+<attribute name="VALUE" x="14.859" y="19.3675" size="1.27" layer="28" rot="MR90"/>
 </element>
 </elements>
@@
 <wire x1="33.9725" y1="24.13" x2="32.9175" y2="22.86" width="0.254" layer="1"/>
 <contactref element="JP1" pad="1"/>
-<wire x1="18.6055" y1="20.32" x2="20.955" y2="18.5175" width="0" layer="19" extent="1-1"/>
+<wire x1="18.161" y1="20.6375" x2="20.955" y2="18.5175" width="0" layer="19" extent="1-1"/>
 </signal>
 <signal name="VCC">
@@
 <wire x1="29.845" y1="31.115" x2="28.79" y2="31.115" width="0.254" layer="1"/>
 <contactref element="JP1" pad="6"/>
-<wire x1="18.8595" y1="33.02" x2="26.6446" y2="29.8196" width="0" layer="19" extent="1-1"/>
+<wire x1="17.907" y1="33.3375" x2="26.6446" y2="29.8196" width="0" layer="19" extent="1-1"/>
 </signal>
 <signal name="BSL_TEST">
@@
 <via x="28.8925" y="29.845" extent="1-16" drill="0.254"/>
 <contactref element="JP1" pad="2"/>
-<wire x1="18.8595" y1="22.86" x2="27.1526" y2="28.8798" width="0" layer="19" extent="1-1"/>
+<wire x1="17.907" y1="23.1775" x2="27.1526" y2="28.8798" width="0" layer="19" extent="1-1"/>
 </signal>
 <signal name="BSL_RX">
 <contactref element="U2" pad="6"/>
 <contactref element="JP1" pad="4"/>
-<wire x1="18.8595" y1="27.94" x2="21.9202" y2="25.654" width="0" layer="19" extent="1-1"/>
+<wire x1="17.907" y1="28.2575" x2="21.9202" y2="25.654" width="0" layer="19" extent="1-1"/>
 </signal>
 <signal name="BSL_TX">
 <contactref element="U2" pad="5"/>
 <contactref element="JP1" pad="5"/>
-<wire x1="21.9202" y1="26.162" x2="18.6055" y2="30.48" width="0" layer="19" extent="1-1"/>
+<wire x1="21.9202" y1="26.162" x2="18.161" y2="30.7975" width="0" layer="19" extent="1-1"/>
 </signal>
 <signal name="XOUT">
@@
 <contactref element="U2" pad="22"/>
 <wire x1="21.9202" y1="24.638" x2="27.1526" y2="21.9202" width="0" layer="19" extent="1-1"/>
-<wire x1="18.6055" y1="25.4" x2="21.9202" y2="24.638" width="0" layer="19" extent="1-1"/>
+<wire x1="18.161" y1="25.7175" x2="21.9202" y2="24.638" width="0" layer="19" extent="1-1"/>
 </signal>
 </signals>
