File: pcb/charliewatch-norf.sch (EAGLE design)
At the start: 84 parts, among them K1 TS-1188E, U2 CC430F5137IRGZR, X1 CRYSTALS-NOGND-IQXC-25

Commit message: routed version of the no-rf variant, with 1 square inch of board area
Parts:
- removed K1: TS-1188E, Seeed-Switch:SMD-BUTTON(2+2P-7X3.5MM-90D)
- added S2: MOMENTARY-SWITCH-SPST-SMD-RIGHT-ANGLE, SparkFun-Switches:MOMENTARY-SWITCH-SPST-SMD-RIGHT-ANGLE
Connections:
- net BUTTON: now also S2.2; no longer K1.2
- net GND: now also S2.1; no longer K1.1
Changed lines of the file:
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@@
 <part name="GND3" library="supply1" deviceset="GND" device=""/>
 <part name="U$1" library="adafruit" deviceset="CR2032" device="SMT"/>
-<part name="K1" library="Seeed-Switch" deviceset="SMD-BUTTON(2+2P-7X3.5MM-90D)" device="" value="TS-1188E"/>
 <part name="TP1" library="testpad" deviceset="PTR1" device="TP10SQ"/>
 <part name="TP2" library="testpad" deviceset="PTR1" device="TP10R"/>
@@
 <part name="TP5" library="testpad" deviceset="PTR1" device="TP10R"/>
 <part name="TP6" library="testpad" deviceset="PTR1" device="TP10R"/>
+<part name="S2" library="SparkFun-Switches" deviceset="MOMENTARY-SWITCH-SPST" device="-SMD-RIGHT-ANGLE"/>
 </parts>
 <sheets>
@@
 <instance part="GND3" gate="1" x="109.22" y="96.52"/>
 <instance part="U$1" gate="G$1" x="20.32" y="22.86"/>
-<instance part="K1" gate="K" x="138.43" y="52.07"/>
 <instance part="TP1" gate="G$1" x="66.04" y="27.94"/>
 <instance part="TP2" gate="G$1" x="68.58" y="25.4"/>
@@
 <instance part="TP5" gate="G$1" x="78.74" y="17.78"/>
 <instance part="TP6" gate="G$1" x="83.82" y="15.24"/>
+<instance part="S2" gate="G$1" x="137.16" y="50.8"/>
 </instances>
 <busses>
@@
 </segment>
 <segment>
-<pinref part="K1" gate="K" pin="1"/>
 <wire x1="132.08" y1="50.8" x2="121.92" y2="50.8" width="0.1524" layer="91"/>
 <label x="119.38" y="50.8" size="1.778" layer="95"/>
+<pinref part="S2" gate="G$1" pin="1"/>
 </segment>
 </net>
@@
 <net name="BUTTON" class="0">
 <segment>
-<pinref part="K1" gate="K" pin="2"/>
-<wire x1="144.78" y1="50.8" x2="152.4" y2="50.8" width="0.1524" layer="91"/>
 <label x="149.86" y="50.8" size="1.778" layer="95"/>
-</segment>
-<segment>
+<pinref part="S2" gate="G$1" pin="2"/>
+<wire x1="142.24" y1="50.8" x2="152.4" y2="50.8" width="0.1524" layer="91"/>
+<junction x="142.24" y="50.8"/>
+</segment>
+<segment>
