File: pcb/charliewatch-bicolor.sch (EAGLE design)
At the start: 79 parts, among them U2 CC430F5137IRGZR, X1 CRYSTALS-NOGND-IQXC-25

Commit message: initial positioning for the bicolor leds
Parts:
- removed D61, D62, D63, D64, D65, D66: APHB1608SYKSURKC, APHB1608SYKSURKC:APHB1608SYKSURKC
- added LED1, LED10, LED11, LED12, LED2, LED3, LED4, LED5, LED6, LED7, LED8, LED9: (no value), led:LEDCHIPLED_0805
Connections:
- removed net N$1: D10G$1.Y_C, D10G$2.R_A, D13G$1.Y_C, D13G$2.R_A, D17G$1.Y_C, D17G$2.R_A, D1G$1.Y_C, D1G$2.R_A, D21G$1.Y_C, D21G$2.R_A, D26G$1.Y_C, D26G$2.R_A, D2G$1.Y_C, D2G$2.R_A, D31G$1.Y_C, D31G$2.R_A, D3G$1.Y_C, D3G$2.R_A, D5G$1.Y_C, D5G$2.R_A, D7G$1.Y_C, D7G$2.R_A
- removed net N$10: D21G$1.Y_A, D21G$2.R_C, D27G$1.Y_A, D27G$2.R_C, D33G$1.Y_A, D33G$2.R_C, D39G$1.Y_A, D39G$2.R_C, D44G$1.Y_A, D44G$2.R_C, D49G$1.Y_A, D49G$2.R_C, D53G$1.Y_A, D53G$2.R_C, D57G$1.Y_A, D57G$2.R_C, D60G$1.Y_A, D60G$2.R_C, D64G$1.Y_C, D64G$2.R_A, D65G$1.Y_C, D65G$2.R_A
- removed net N$11: D26G$1.Y_A, D26G$2.R_C, D32G$1.Y_A, D32G$2.R_C, D38G$1.Y_A, D38G$2.R_C, D43G$1.Y_A, D43G$2.R_C, D48G$1.Y_A, D48G$2.R_C, D52G$1.Y_A, D52G$2.R_C, D56G$1.Y_A, D56G$2.R_C, D59G$1.Y_A, D59G$2.R_C, D62G$1.Y_A, D62G$2.R_C, D64G$1.Y_A, D64G$2.R_C, D66G$1.Y_C, D66G$2.R_A
- removed net N$12: D31G$1.Y_A, D31G$2.R_C, D37G$1.Y_A, D37G$2.R_C, D42G$1.Y_A, D42G$2.R_C, D47G$1.Y_A, D47G$2.R_C, D51G$1.Y_A, D51G$2.R_C, D55G$1.Y_A, D55G$2.R_C, D58G$1.Y_A, D58G$2.R_C, D61G$1.Y_A, D61G$2.R_C, D63G$1.Y_A, D63G$2.R_C, D65G$1.Y_A, D65G$2.R_C, D66G$1.Y_A, D66G$2.R_C
- removed net N$2: D11G$1.Y_C, D11G$2.R_A, D14G$1.Y_C, D14G$2.R_A, D18G$1.Y_C, D18G$2.R_A, D1G$1.Y_A, D1G$2.R_C, D22G$1.Y_C, D22G$2.R_A, D27G$1.Y_C, D27G$2.R_A, D32G$1.Y_C, D32G$2.R_A, D37G$1.Y_C, D37G$2.R_A, D4G$1.Y_C, D4G$2.R_A, D6G$1.Y_C, D6G$2.R_A, D8G$1.Y_C, D8G$2.R_A
- removed net N$3: D12G$1.Y_C, D12G$2.R_A, D15G$1.Y_C, D15G$2.R_A, D19G$1.Y_C, D19G$2.R_A, D23G$1.Y_C, D23G$2.R_A, D28G$1.Y_C, D28G$2.R_A, D2G$1.Y_A, D2G$2.R_C, D33G$1.Y_C, D33G$2.R_A, D38G$1.Y_C, D38G$2.R_A, D42G$1.Y_C, D42G$2.R_A, D4G$1.Y_A, D4G$2.R_C, D9G$1.Y_C, D9G$2.R_A
- removed net N$4: D16G$1.Y_C, D16G$2.R_A, D20G$1.Y_C, D20G$2.R_A, D24G$1.Y_C, D24G$2.R_A, D29G$1.Y_C, D29G$2.R_A, D34G$1.Y_C, D34G$2.R_A, D39G$1.Y_C, D39G$2.R_A, D3G$1.Y_A, D3G$2.R_C, D43G$1.Y_C, D43G$2.R_A, D47G$1.Y_C, D47G$2.R_A, D6G$1.Y_A, D6G$2.R_C, D9G$1.Y_A, D9G$2.R_C
- removed net N$5: D12G$1.Y_A, D12G$2.R_C, D16G$1.Y_A, D16G$2.R_C, D25G$1.Y_C, D25G$2.R_A, D30G$1.Y_C, D30G$2.R_A, D35G$1.Y_C, D35G$2.R_A, D40G$1.Y_C, D40G$2.R_A, D44G$1.Y_C, D44G$2.R_A, D48G$1.Y_C, D48G$2.R_A, D51G$1.Y_C, D51G$2.R_A, D5G$1.Y_A, D5G$2.R_C, D8G$1.Y_A, D8G$2.R_C
- removed net N$6: D11G$1.Y_A, D11G$2.R_C, D15G$1.Y_A, D15G$2.R_C, D20G$1.Y_A, D20G$2.R_C, D25G$1.Y_A, D25G$2.R_C, D36G$1.Y_C, D36G$2.R_A, D41G$1.Y_C, D41G$2.R_A, D45G$1.Y_C, D45G$2.R_A, D49G$1.Y_C, D49G$2.R_A, D52G$1.Y_C, D52G$2.R_A, D55G$1.Y_C, D55G$2.R_A, D7G$1.Y_A, D7G$2.R_C
- removed net N$7: D10G$1.Y_A, D10G$2.R_C, D14G$1.Y_A, D14G$2.R_C, D19G$1.Y_A, D19G$2.R_C, D24G$1.Y_A, D24G$2.R_C, D30G$1.Y_A, D30G$2.R_C, D36G$1.Y_A, D36G$2.R_C, D46G$1.Y_C, D46G$2.R_A, D50G$1.Y_C, D50G$2.R_A, D53G$1.Y_C, D53G$2.R_A, D56G$1.Y_C, D56G$2.R_A, D58G$1.Y_C, D58G$2.R_A
- removed net N$8: D13G$1.Y_A, D13G$2.R_C, D18G$1.Y_A, D18G$2.R_C, D23G$1.Y_A, D23G$2.R_C, D29G$1.Y_A, D29G$2.R_C, D35G$1.Y_A, D35G$2.R_C, D41G$1.Y_A, D41G$2.R_C, D46G$1.Y_A, D46G$2.R_C, D54G$1.Y_C, D57G$1.Y_C, D57G$2.R_A, D59G$1.Y_C, D59G$2.R_A, D61G$1.Y_C, D61G$2.R_A
- removed net N$9: D17G$1.Y_A, D17G$2.R_C, D22G$1.Y_A, D22G$2.R_C, D28G$1.Y_A, D28G$2.R_C, D34G$1.Y_A, D34G$2.R_C, D40G$1.Y_A, D40G$2.R_C, D45G$1.Y_A, D45G$2.R_C, D50G$1.Y_A, D50G$2.R_C, D54G$1.Y_A, D54G$2.R_C, D60G$1.Y_C, D60G$2.R_A, D62G$1.Y_C, D62G$2.R_A, D63G$1.Y_C, D63G$2.R_A
- removed net P3.5: U2.P3.5/PM_TA0CCR4A
- removed net P3.6: U2.P3.6/PM_RFGDO1
- removed net P3.7: U2.P3.7/PM_SMCLK
- new net B10: D26G$1.Y_A, D26G$2.R_C, D32G$1.Y_A, D32G$2.R_C, D38G$1.Y_A, D38G$2.R_C, D43G$1.Y_A, D43G$2.R_C, D48G$1.Y_A, D48G$2.R_C, D52G$1.Y_A, D52G$2.R_C, D55G$1.Y_A, D55G$2.R_C, D56G$1.Y_A, D56G$2.R_C, D58G$1.Y_A, D58G$2.R_C, D59G$1.Y_A, D59G$2.R_C, LED7.A, U2.P2.2/PM_TA1CCR1A/CB2/A2
- new net B11: D31G$1.Y_A, D31G$2.R_C, D37G$1.Y_A, D37G$2.R_C, D42G$1.Y_A, D42G$2.R_C, D47G$1.Y_A, D47G$2.R_C, D51G$1.Y_A, D51G$2.R_C, LED1.A, LED2.A, LED3.A, LED4.A, LED5.A, LED6.A, U2.P2.3/PM_TA1CCR2A/CB3/A3
- new net B9: D21G$1.Y_A, D21G$2.R_C, D27G$1.Y_A, D27G$2.R_C, D33G$1.Y_A, D33G$2.R_C, D39G$1.Y_A, D39G$2.R_C, D44G$1.Y_A, D44G$2.R_C, D49G$1.Y_A, D49G$2.R_C, D53G$1.Y_A, D53G$2.R_C, D57G$1.Y_A, D57G$2.R_C, D58G$1.Y_C, D58G$2.R_A, D60G$1.Y_A, D60G$2.R_C, LED8.A, U2.P2.1/PM_TA1CCR0A/CB1/A1
- net B0: now also D10G$1.Y_C, D10G$2.R_A, D13G$1.Y_C, D13G$2.R_A, D17G$1.Y_C, D17G$2.R_A, D1G$1.Y_C, D1G$2.R_A, D21G$1.Y_C, D21G$2.R_A, D26G$1.Y_C, D26G$2.R_A, D2G$1.Y_C, D2G$2.R_A, D31G$1.Y_C, D31G$2.R_A, D3G$1.Y_C, D3G$2.R_A, D5G$1.Y_C, D5G$2.R_A, D7G$1.Y_C, D7G$2.R_A
- net B1: now also D11G$1.Y_C, D11G$2.R_A, D14G$1.Y_C, D14G$2.R_A, D18G$1.Y_C, D18G$2.R_A, D1G$1.Y_A, D1G$2.R_C, D22G$1.Y_C, D22G$2.R_A, D27G$1.Y_C, D27G$2.R_A, D32G$1.Y_C, D32G$2.R_A, D37G$1.Y_C, D37G$2.R_A, D4G$1.Y_C, D4G$2.R_A, D6G$1.Y_C, D6G$2.R_A, D8G$1.Y_C, D8G$2.R_A
- net B2: now also D12G$1.Y_C, D12G$2.R_A, D15G$1.Y_C, D15G$2.R_A, D19G$1.Y_C, D19G$2.R_A, D23G$1.Y_C, D23G$2.R_A, D28G$1.Y_C, D28G$2.R_A, D2G$1.Y_A, D2G$2.R_C, D33G$1.Y_C, D33G$2.R_A, D38G$1.Y_C, D38G$2.R_A, D42G$1.Y_C, D42G$2.R_A, D4G$1.Y_A, D4G$2.R_C, D9G$1.Y_C, D9G$2.R_A
- net B3: now also D16G$1.Y_C, D16G$2.R_A, D20G$1.Y_C, D20G$2.R_A, D24G$1.Y_C, D24G$2.R_A, D29G$1.Y_C, D29G$2.R_A, D34G$1.Y_C, D34G$2.R_A, D39G$1.Y_C, D39G$2.R_A, D3G$1.Y_A, D3G$2.R_C, D43G$1.Y_C, D43G$2.R_A, D47G$1.Y_C, D47G$2.R_A, D6G$1.Y_A, D6G$2.R_C, D9G$1.Y_A, D9G$2.R_C
- net B4: now also D12G$1.Y_A, D12G$2.R_C, D16G$1.Y_A, D16G$2.R_C, D25G$1.Y_C, D25G$2.R_A, D30G$1.Y_C, D30G$2.R_A, D35G$1.Y_C, D35G$2.R_A, D40G$1.Y_C, D40G$2.R_A, D44G$1.Y_C, D44G$2.R_A, D48G$1.Y_C, D48G$2.R_A, D51G$1.Y_C, D51G$2.R_A, D5G$1.Y_A, D5G$2.R_C, D8G$1.Y_A, D8G$2.R_C
- net B5: now also D11G$1.Y_A, D11G$2.R_C, D15G$1.Y_A, D15G$2.R_C, D20G$1.Y_A, D20G$2.R_C, D25G$1.Y_A, D25G$2.R_C, D36G$1.Y_C, D36G$2.R_A, D41G$1.Y_C, D41G$2.R_A, D45G$1.Y_C, D45G$2.R_A, D49G$1.Y_C, D49G$2.R_A, D52G$1.Y_C, D52G$2.R_A, D7G$1.Y_A, D7G$2.R_C, LED1.C, LED12.A, U2.P3.5/PM_TA0CCR4A; no longer U2.P2.0/PM_CBOUT1/PM_TA1CLK/CB0/A0
- net B6: now also D10G$1.Y_A, D10G$2.R_C, D14G$1.Y_A, D14G$2.R_C, D19G$1.Y_A, D19G$2.R_C, D24G$1.Y_A, D24G$2.R_C, D30G$1.Y_A, D30G$2.R_C, D36G$1.Y_A, D36G$2.R_C, D46G$1.Y_C, D46G$2.R_A, D50G$1.Y_C, D50G$2.R_A, D53G$1.Y_C, D53G$2.R_A, D56G$1.Y_C, D56G$2.R_A, LED11.A, LED2.C, U2.P3.6/PM_RFGDO1; no longer U2.P2.1/PM_TA1CCR0A/CB1/A1
- net B7: now also D13G$1.Y_A, D13G$2.R_C, D18G$1.Y_A, D18G$2.R_C, D23G$1.Y_A, D23G$2.R_C, D29G$1.Y_A, D29G$2.R_C, D35G$1.Y_A, D35G$2.R_C, D41G$1.Y_A, D41G$2.R_C, D46G$1.Y_A, D46G$2.R_C, D54G$1.Y_C, D57G$1.Y_C, D57G$2.R_A, D59G$1.Y_C, D59G$2.R_A, LED10.A, U2.P3.7/PM_SMCLK; no longer U2.P2.2/PM_TA1CCR1A/CB2/A2
- net B8: now also D17G$1.Y_A, D17G$2.R_C, D22G$1.Y_A, D22G$2.R_C, D28G$1.Y_A, D28G$2.R_C, D34G$1.Y_A, D34G$2.R_C, D40G$1.Y_A, D40G$2.R_C, D45G$1.Y_A, D45G$2.R_C, D50G$1.Y_A, D50G$2.R_C, D54G$1.Y_A, D54G$2.R_C, D55G$1.Y_C, D55G$2.R_A, D60G$1.Y_C, D60G$2.R_A, LED9.A, U2.P2.0/PM_CBOUT1/PM_TA1CLK/CB0/A0; no longer U2.P2.3/PM_TA1CCR2A/CB3/A3

Commit message: change to through-hole cr2032 and hack up the layout
Parts:
- U$1: device adafruit:CR2032SMT -> adafruit:CR2032THM
Changed lines of the file:
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@@
 <grid distance="0.1" unitdist="inch" unit="inch" style="lines" multiple="1" display="no" altdistance="0.01" altunitdist="inch" altunit="inch"/>
 <layers>
-<layer number="1" name="Top" color="4" fill="1" visible="no" active="no"/>
-<layer number="2" name="Route2" color="1" fill="3" visible="no" active="no"/>
-<layer number="3" name="Route3" color="4" fill="3" visible="no" active="no"/>
-<layer number="14" name="Route14" color="1" fill="6" visible="no" active="no"/>
-<layer number="15" name="Route15" color="4" fill="6" visible="no" active="no"/>
-<layer number="16" name="Bottom" color="1" fill="1" visible="no" active="no"/>
-<layer number="17" name="Pads" color="2" fill="1" visible="no" active="no"/>
-<layer number="18" name="Vias" color="2" fill="1" visible="no" active="no"/>
-<layer number="19" name="Unrouted" color="6" fill="1" visible="no" active="no"/>
-<layer number="20" name="Dimension" color="15" fill="1" visible="no" active="no"/>
-<layer number="21" name="tPlace" color="7" fill="1" visible="no" active="no"/>
-<layer number="22" name="bPlace" color="7" fill="1" visible="no" active="no"/>
-<layer number="23" name="tOrigins" color="15" fill="1" visible="no" active="no"/>
-<layer number="24" name="bOrigins" color="15" fill="1" visible="no" active="no"/>
-<layer number="25" name="tNames" color="7" fill="1" visible="no" active="no"/>
-<layer number="26" name="bNames" color="7" fill="1" visible="no" active="no"/>
-<layer number="27" name="tValues" color="7" fill="1" visible="no" active="no"/>
-<layer number="28" name="bValues" color="7" fill="1" visible="no" active="no"/>
+<layer number="1" name="Top" color="4" fill="1" visible="yes" active="no"/>
+<layer number="2" name="Route2" color="1" fill="3" visible="yes" active="no"/>
+<layer number="3" name="Route3" color="4" fill="3" visible="yes" active="no"/>
+<layer number="14" name="Route14" color="1" fill="6" visible="yes" active="no"/>
+<layer number="15" name="Route15" color="4" fill="6" visible="yes" active="no"/>
+<layer number="16" name="Bottom" color="1" fill="1" visible="yes" active="no"/>
+<layer number="17" name="Pads" color="2" fill="1" visible="yes" active="no"/>
+<layer number="18" name="Vias" color="2" fill="1" visible="yes" active="no"/>
+<layer number="19" name="Unrouted" color="6" fill="1" visible="yes" active="no"/>
+<layer number="20" name="Dimension" color="15" fill="1" visible="yes" active="no"/>
+<layer number="21" name="tPlace" color="7" fill="1" visible="yes" active="no"/>
+<layer number="22" name="bPlace" color="7" fill="1" visible="yes" active="no"/>
+<layer number="23" name="tOrigins" color="15" fill="1" visible="yes" active="no"/>
+<layer number="24" name="bOrigins" color="15" fill="1" visible="yes" active="no"/>
+<layer number="25" name="tNames" color="7" fill="1" visible="yes" active="no"/>
+<layer number="26" name="bNames" color="7" fill="1" visible="yes" active="no"/>
+<layer number="27" name="tValues" color="7" fill="1" visible="yes" active="no"/>
+<layer number="28" name="bValues" color="7" fill="1" visible="yes" active="no"/>
 <layer number="29" name="tStop" color="7" fill="3" visible="no" active="no"/>
 <layer number="30" name="bStop" color="7" fill="6" visible="no" active="no"/>
@@
 <layer number="35" name="tGlue" color="7" fill="4" visible="no" active="no"/>
 <layer number="36" name="bGlue" color="7" fill="5" visible="no" active="no"/>
-<layer number="37" name="tTest" color="7" fill="1" visible="no" active="no"/>
-<layer number="38" name="bTest" color="7" fill="1" visible="no" active="no"/>
+<layer number="37" name="tTest" color="7" fill="1" visible="yes" active="no"/>
+<layer number="38" name="bTest" color="7" fill="1" visible="yes" active="no"/>
 <layer number="39" name="tKeepout" color="4" fill="11" visible="no" active="no"/>
 <layer number="40" name="bKeepout" color="1" fill="11" visible="no" active="no"/>
@@
 <layer number="44" name="Drills" color="7" fill="1" visible="no" active="no"/>
 <layer number="45" name="Holes" color="7" fill="1" visible="no" active="no"/>
-<layer number="46" name="Milling" color="3" fill="1" visible="no" active="no"/>
-<layer number="47" name="Measures" color="7" fill="1" visible="no" active="no"/>
-<layer number="48" name="Document" color="7" fill="1" visible="no" active="no"/>
-<layer number="49" name="Reference" color="7" fill="1" visible="no" active="no"/>
-<layer number="50" name="dxf" color="7" fill="1" visible="no" active="no"/>
-<layer number="51" name="tDocu" color="7" fill="1" visible="no" active="no"/>
-<layer number="52" name="bDocu" color="7" fill="1" visible="no" active="no"/>
-<layer number="53" name="tPadExt" color="7" fill="1" visible="no" active="no"/>
-<layer number="54" name="bPadExt" color="1" fill="1" visible="no" active="no"/>
-<layer number="56" name="wert" color="7" fill="1" visible="no" active="no"/>
-<layer number="57" name="tCAD" color="7" fill="1" visible="no" active="no"/>
-<layer number="59" name="tCarbon" color="7" fill="1" visible="no" active="no"/>
-<layer number="60" name="bCarbon" color="7" fill="1" visible="no" active="no"/>
+<layer number="46" name="Milling" color="3" fill="1" visible="yes" active="no"/>
+<layer number="47" name="Measures" color="7" fill="1" visible="yes" active="no"/>
+<layer number="48" name="Document" color="7" fill="1" visible="yes" active="no"/>
+<layer number="49" name="Reference" color="7" fill="1" visible="yes" active="no"/>
+<layer number="50" name="dxf" color="7" fill="1" visible="yes" active="no"/>
+<layer number="51" name="tDocu" color="7" fill="1" visible="yes" active="no"/>
+<layer number="52" name="bDocu" color="7" fill="1" visible="yes" active="no"/>
+<layer number="53" name="tPadExt" color="7" fill="1" visible="yes" active="no"/>
+<layer number="54" name="bPadExt" color="1" fill="1" visible="yes" active="no"/>
+<layer number="56" name="wert" color="7" fill="1" visible="yes" active="no"/>
+<layer number="57" name="tCAD" color="7" fill="1" visible="yes" active="no"/>
+<layer number="59" name="tCarbon" color="7" fill="1" visible="yes" active="no"/>
+<layer number="60" name="bCarbon" color="7" fill="1" visible="yes" active="no"/>
 <layer number="90" name="Modules" color="5" fill="1" visible="yes" active="yes"/>
 <layer number="91" name="Nets" color="2" fill="1" visible="yes" active="yes"/>
@@
 <part name="L1" library="rcl" deviceset="R-EU_" device="R0603"/>
 <part name="GND3" library="supply1" deviceset="GND" device=""/>
-<part name="U$1" library="adafruit" deviceset="CR2032" device="SMT"/>
+<part name="U$1" library="adafruit" deviceset="CR2032" device="THM"/>
 <part name="TP1" library="testpad" deviceset="PTR1" device="TP10SQ"/>
 <part name="TP2" library="testpad" deviceset="PTR1" device="TP10R"/>
